File: FOC.kicad_pcb (KiCad board)
At the start: 4 copper layers, 185.8 x 69.2 mm, 80 parts, among them IC1 STM32C071KBT6, IC2 DRV8300DPWR, IC3 TPS54308DDCT, IC4 TLV7034QPWRQ1, J1 STLINK_INTERFACE, J2 PWR_PWM_INPUT, J3 MOTOR_OUTPUT, Q1 SUM60020E-GE3, Q2 SUM60020E-GE3, Q3 SUM60020E-GE3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

Commit message: Final Push
Parts:
- moved C6 2.07 mm to (120.0, 109.5)
- moved C2 1.82 mm to (124.0, 109.5)
Connections:
- L1 pad 1: Net-(IC3-BOOT) -> Net-(IC3-SW)
Routing:
- net VDD: track 159.7 -> 23.8 mm, vias 15 -> 46
- net GND: track 162.4 -> 99.4 mm, vias 24 -> 46
- net 3.3V: track 77.8 -> 63.5 mm, vias 8 -> 9
- net Net-(IC3-SW): track 5.41 -> 14.2 mm
- net Net-(IC3-BOOT): track 11.4 -> 3.44 mm
- added copper zone on F.Cu, net 3.3V
- added copper zone on F.Cu, net GND
- added copper zone on F.Cu, net VDD
Other:
- board text added: "3.3V"
- board text added: "NRST"
- board text added: "Rishit Arora ESC PCB v1.0"
- board text added: "SWCLK"
- board text added: "SWDIO"
