File: FOC.kicad_sch (KiCad schematic)
At the start: 76 parts, among them IC1 STM32C071KBT6, IC2 DRV8300DPWR, IC3 TPS54308DDCT, IC4 TLV7034QPWRQ1, J1 STLINK_INTERFACE, J2 PWR_PWM_INPUT, J3 MOTOR_OUTPUT, Q1 SUM60020E-GE3, Q2 SUM60020E-GE3, Q3 SUM60020E-GE3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

Commit message: Final Push
Connections:
- net at C11.1, IC3.6 (BOOT): no longer L1.1
- net at C11.2, IC3.2 (SW): now also L1.1
